File: hardware/cmpe195_laztech/laztech.brd (EAGLE design)
At the start: 68.6 x 61 mm, 21 parts

Commit message: Added pin directions and resistor symbols.
Parts:
- added R1, R2, R3, R4, R5, R6, R7: RES, laztech_parts:R2012
- moved U$8 7.73 mm to (22.9, 12.7)
- moved C13 6.48 mm to (19.1, 7.62)
Connections:
- new net N$34: R2.1, R3.2, U$8.2, U$8.3, U$8.6, U$8.7
- new net N$35: R5.1, U$1.20
- new net N$38: R6.1, U$2.17
- new net N$40: R7.1, U$2.20
- new net N$9: R4.1, U$1.17
- new net VREF: R1.2, R2.2, R3.1, U$1.12, U$2.12, U$8.4
- net GND: now also R1.1, R4.2, R5.2, R6.2, R7.2
Changed lines of the file:
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@@
 <element name="C11" library="laztech_parts" package="C2012" value="" x="41.91" y="24.13" rot="R180"/>
 <element name="C12" library="laztech_parts" package="C2012" value="" x="15.24" y="43.18" rot="R90"/>
-<element name="U$8" library="laztech_parts" package="SOIC-8" value="LM317" x="24.13" y="5.08"/>
-<element name="C13" library="laztech_parts" package="C2012" value="" x="20.32" y="1.27" rot="R180"/>
+<element name="U$8" library="laztech_parts" package="SOIC-8" value="LM317" x="22.86" y="12.7"/>
+<element name="C13" library="laztech_parts" package="C2012" value="" x="19.05" y="7.62" rot="R180"/>
+<element name="R1" library="laztech_parts" package="R2012" value="RES" x="25.4" y="5.08" rot="R180"/>
+<element name="R2" library="laztech_parts" package="R2012" value="RES" x="22.86" y="7.62"/>
+<element name="R3" library="laztech_parts" package="R2012" value="RES" x="21.59" y="5.08" rot="R180"/>
+<element name="R4" library="laztech_parts" package="R2012" value="RES" x="49.53" y="33.02" rot="R90"/>
+<element name="R5" library="laztech_parts" package="R2012" value="RES" x="43.18" y="33.02" rot="R90"/>
+<element name="R6" library="laztech_parts" package="R2012" value="RES" x="22.86" y="35.56"/>
+<element name="R7" library="laztech_parts" package="R2012" value="RES" x="22.86" y="41.91"/>
 </elements>
 <signals>
@@
 <contactref element="C3" pad="2"/>
 <contactref element="C13" pad="2"/>
+<contactref element="R7" pad="2"/>
+<contactref element="R6" pad="2"/>
+<contactref element="R5" pad="2"/>
+<contactref element="R4" pad="2"/>
+<contactref element="R1" pad="1"/>
 <wire x1="48.885" y1="50.84" x2="64.41" y2="48.26" width="0" layer="19" extent="1-1"/>
-<wire x1="55.88" y1="25.71" x2="64.41" y2="48.26" width="0" layer="19" extent="1-1"/>
-<wire x1="51.835" y1="20.83" x2="55.88" y2="25.71" width="0" layer="19" extent="1-1"/>
-<wire x1="48.26" y1="17.78" x2="51.835" y2="20.83" width="0" layer="19" extent="1-1"/>
+<wire x1="49.53" y1="34.02" x2="48.885" y2="50.84" width="0" layer="19" extent="1-1"/>
+<wire x1="43.18" y1="34.02" x2="49.53" y2="34.02" width="0" layer="19" extent="1-1"/>
+<wire x1="40.91" y1="24.13" x2="43.18" y2="34.02" width="0" layer="19" extent="1-1"/>
+<wire x1="44.685" y1="20.83" x2="40.91" y2="24.13" width="0" layer="19" extent="1-1"/>
+<wire x1="48.26" y1="17.78" x2="44.685" y2="20.83" width="0" layer="19" extent="1-1"/>
 <wire x1="49.235" y1="14.73" x2="48.26" y2="17.78" width="0" layer="19" extent="1-1"/>
-<wire x1="44.685" y1="20.83" x2="48.26" y2="17.78" width="0" layer="19" extent="1-1"/>
+<wire x1="51.835" y1="20.83" x2="48.26" y2="17.78" width="0" layer="19" extent="1-1"/>
 <wire x1="46.99" y1="10.43" x2="49.235" y2="14.73" width="0" layer="19" extent="1-1"/>
-<wire x1="40.91" y1="24.13" x2="44.685" y2="20.83" width="0" layer="19" extent="1-1"/>
 <wire x1="52.07" y1="10.43" x2="46.99" y2="10.43" width="0" layer="19" extent="1-1"/>
+<wire x1="55.88" y1="25.71" x2="51.835" y2="20.83" width="0" layer="19" extent="1-1"/>
 <wire x1="61.87" y1="10.16" x2="52.07" y2="10.43" width="0" layer="19" extent="1-1"/>
-<wire x1="16.82" y1="29.21" x2="40.91" y2="24.13" width="0" layer="19" extent="1-1"/>
-<wire x1="11.94" y1="33.255" x2="16.82" y2="29.21" width="0" layer="19" extent="1-1"/>
-<wire x1="8.89" y1="36.83" x2="11.94" y2="33.255" width="0" layer="19" extent="1-1"/>
+<wire x1="23.86" y1="35.56" x2="43.18" y2="34.02" width="0" layer="19" extent="1-1"/>
+<wire x1="23.86" y1="41.91" x2="23.86" y2="35.56" width="0" layer="19" extent="1-1"/>
+<wire x1="15.24" y1="44.18" x2="23.86" y2="41.91" width="0" layer="19" extent="1-1"/>
+<wire x1="11.94" y1="40.405" x2="15.24" y2="44.18" width="0" layer="19" extent="1-1"/>
+<wire x1="8.89" y1="36.83" x2="11.94" y2="40.405" width="0" layer="19" extent="1-1"/>
 <wire x1="5.84" y1="35.855" x2="8.89" y2="36.83" width="0" layer="19" extent="1-1"/>
-<wire x1="11.94" y1="40.405" x2="8.89" y2="36.83" width="0" layer="19" extent="1-1"/>
+<wire x1="11.94" y1="33.255" x2="8.89" y2="36.83" width="0" layer="19" extent="1-1"/>
 <wire x1="1.54" y1="38.1" x2="5.84" y2="35.855" width="0" layer="19" extent="1-1"/>
-<wire x1="15.24" y1="44.18" x2="11.94" y2="40.405" width="0" layer="19" extent="1-1"/>
 <wire x1="1.54" y1="33.02" x2="1.54" y2="38.1" width="0" layer="19" extent="1-1"/>
+<wire x1="16.82" y1="29.21" x2="11.94" y2="33.255" width="0" layer="19" extent="1-1"/>
 <wire x1="17.22" y1="50.8" x2="15.24" y2="44.18" width="0" layer="19" extent="1-1"/>
 <wire x1="2.54" y1="50.08" x2="1.54" y2="38.1" width="0" layer="19" extent="1-1"/>
-<wire x1="19.32" y1="1.27" x2="16.82" y2="29.21" width="0" layer="19" extent="1-1"/>
+<wire x1="26.4" y1="5.08" x2="46.99" y2="10.43" width="0" layer="19" extent="1-1"/>
+<wire x1="18.05" y1="7.62" x2="26.4" y2="5.08" width="0" layer="19" extent="1-1"/>
 </signal>
 <signal name="+3V3">
@@
 <wire x1="50.535" y1="14.73" x2="64.41" y2="50.8" width="0" layer="19" extent="1-1"/>
 <wire x1="52.07" y1="12.43" x2="50.535" y2="14.73" width="0" layer="19" extent="1-1"/>
-<wire x1="3.54" y1="33.02" x2="50.535" y2="14.73" width="0" layer="19" extent="1-1"/>
-<wire x1="5.84" y1="34.555" x2="3.54" y2="33.02" width="0" layer="19" extent="1-1"/>
+<wire x1="5.84" y1="34.555" x2="50.535" y2="14.73" width="0" layer="19" extent="1-1"/>
+<wire x1="3.54" y1="33.02" x2="5.84" y2="34.555" width="0" layer="19" extent="1-1"/>
 </signal>
 <signal name="+5V">
@@
 <contactref element="U$2" pad="1"/>
 <contactref element="C6" pad="1"/>
-<wire x1="3.81" y1="44.18" x2="5.84" y2="40.405" width="0" layer="19" extent="1-1"/>
+<wire x1="5.84" y1="40.405" x2="3.81" y2="44.18" width="0" layer="19" extent="1-1"/>
 </signal>
 <signal name="N$28">
 <contactref element="C6" pad="2"/>
 <contactref element="U$2" pad="2"/>
-<wire x1="3.81" y1="42.18" x2="5.84" y2="39.755" width="0" layer="19" extent="1-1"/>
+<wire x1="5.84" y1="39.755" x2="3.81" y2="42.18" width="0" layer="19" extent="1-1"/>
 </signal>
 <signal name="N$29">
@@
 <wire x1="21.18" y1="50.8" x2="15.24" y2="42.18" width="0" layer="19" extent="1-1"/>
 <wire x1="1.27" y1="42.91" x2="11.94" y2="38.455" width="0" layer="19" extent="1-1"/>
-<wire x1="22.505" y1="2.03" x2="23.82" y2="29.21" width="0" layer="19" extent="1-1"/>
-<wire x1="21.32" y1="1.27" x2="22.505" y2="2.03" width="0" layer="19" extent="1-1"/>
+<wire x1="20.955" y1="10" x2="23.82" y2="29.21" width="0" layer="19" extent="1-1"/>
+<wire x1="20.05" y1="7.62" x2="20.955" y2="10" width="0" layer="19" extent="1-1"/>
+</signal>
+<signal name="N$34">
+<contactref element="U$8" pad="3"/>
+<contactref element="U$8" pad="6"/>
+<contactref element="U$8" pad="7"/>
+<contactref element="U$8" pad="2"/>
+<contactref element="R2" pad="1"/>
+<contactref element="R3" pad="2"/>
+<wire x1="23.495" y1="15.4" x2="22.225" y2="15.4" width="0" layer="19" extent="1-1"/>
+<wire x1="23.495" y1="10" x2="23.495" y2="15.4" width="0" layer="19" extent="1-1"/>
+<wire x1="22.225" y1="10" x2="23.495" y2="10" width="0" layer="19" extent="1-1"/>
+<wire x1="21.86" y1="7.62" x2="22.225" y2="10" width="0" layer="19" extent="1-1"/>
+<wire x1="20.59" y1="5.08" x2="21.86" y2="7.62" width="0" layer="19" extent="1-1"/>
+</signal>
+<signal name="VREF">
+<contactref element="R3" pad="1"/>
+<contactref element="U$8" pad="4"/>
+<contactref element="R1" pad="2"/>
+<contactref element="R2" pad="2"/>
+<contactref element="U$2" pad="12"/>
+<contactref element="U$1" pad="12"/>
+<wire x1="23.86" y1="7.62" x2="51.835" y2="14.73" width="0" layer="19" extent="1-1"/>
+<wire x1="24.765" y1="10" x2="23.86" y2="7.62" width="0" layer="19" extent="1-1"/>
+<wire x1="24.4" y1="5.08" x2="23.86" y2="7.62" width="0" layer="19" extent="1-1"/>
+<wire x1="22.59" y1="5.08" x2="24.4" y2="5.08" width="0" layer="19" extent="1-1"/>
+<wire x1="5.84" y1="33.255" x2="24.765" y2="10" width="0" layer="19" extent="1-1"/>
+</signal>
+<signal name="N$9">
+<contactref element="U$1" pad="17"/>
+<contactref element="R4" pad="1"/>
+<wire x1="49.235" y1="20.83" x2="49.53" y2="32.02" width="0" layer="19" extent="1-1"/>
+</signal>
+<signal name="N$35">
+<contactref element="U$1" pad="20"/>
+<contactref element="R5" pad="1"/>
+<wire x1="47.285" y1="20.83" x2="43.18" y2="32.02" width="0" layer="19" extent="1-1"/>
+</signal>
+<signal name="N$38">
+<contactref element="U$2" pad="17"/>
+<contactref element="R6" pad="1"/>
+<wire x1="11.94" y1="35.855" x2="21.86" y2="35.56" width="0" layer="19" extent="1-1"/>
+</signal>
+<signal name="N$40">
+<contactref element="U$2" pad="20"/>
+<contactref element="R7" pad="1"/>
+<wire x1="11.94" y1="37.805" x2="21.86" y2="41.91" width="0" layer="19" extent="1-1"/>
 </signal>
 </signals>

Commit message: Added resistor packages.
Parts:
- R1, R2, R3: value RES -> RES2012
- R4, R5, R6, R7: value RES -> RES6432; device laztech_parts:R2012 -> laztech_parts:R6432
- moved R1 2.84 mm to (26.7, 7.62)
- moved C13 2.84 mm to (17.8, 10.2)
- moved R3 1.27 mm to (22.9, 5.08)
Changed lines of the file:
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@@
 <element name="C12" library="laztech_parts" package="C2012" value="" x="15.24" y="43.18" rot="R90"/>
 <element name="U$8" library="laztech_parts" package="SOIC-8" value="LM317" x="22.86" y="12.7"/>
-<element name="C13" library="laztech_parts" package="C2012" value="" x="19.05" y="7.62" rot="R180"/>
-<element name="R1" library="laztech_parts" package="R2012" value="RES" x="25.4" y="5.08" rot="R180"/>
-<element name="R2" library="laztech_parts" package="R2012" value="RES" x="22.86" y="7.62"/>
-<element name="R3" library="laztech_parts" package="R2012" value="RES" x="21.59" y="5.08" rot="R180"/>
-<element name="R4" library="laztech_parts" package="R2012" value="RES" x="49.53" y="33.02" rot="R90"/>
-<element name="R5" library="laztech_parts" package="R2012" value="RES" x="43.18" y="33.02" rot="R90"/>
-<element name="R6" library="laztech_parts" package="R2012" value="RES" x="22.86" y="35.56"/>
-<element name="R7" library="laztech_parts" package="R2012" value="RES" x="22.86" y="41.91"/>
+<element name="C13" library="laztech_parts" package="C2012" value="" x="17.78" y="10.16" rot="R180"/>
+<element name="R1" library="laztech_parts" package="R2012" value="RES2012" x="26.67" y="7.62" rot="R180"/>
+<element name="R2" library="laztech_parts" package="R2012" value="RES2012" x="22.86" y="7.62"/>
+<element name="R3" library="laztech_parts" package="R2012" value="RES2012" x="22.86" y="5.08" rot="R180"/>
+<element name="R4" library="laztech_parts" package="R6432" value="RES6432" x="49.53" y="33.02" rot="R90"/>
+<element name="R5" library="laztech_parts" package="R6432" value="RES6432" x="43.18" y="33.02" rot="R90"/>
+<element name="R6" library="laztech_parts" package="R6432" value="RES6432" x="22.86" y="35.56"/>
+<element name="R7" library="laztech_parts" package="R6432" value="RES6432" x="22.86" y="41.91"/>
 </elements>
 <signals>
@@
 <contactref element="R1" pad="1"/>
 <wire x1="48.885" y1="50.84" x2="64.41" y2="48.26" width="0" layer="19" extent="1-1"/>
-<wire x1="49.53" y1="34.02" x2="48.885" y2="50.84" width="0" layer="19" extent="1-1"/>
-<wire x1="43.18" y1="34.02" x2="49.53" y2="34.02" width="0" layer="19" extent="1-1"/>
-<wire x1="40.91" y1="24.13" x2="43.18" y2="34.02" width="0" layer="19" extent="1-1"/>
+<wire x1="49.53" y1="36.27" x2="48.885" y2="50.84" width="0" layer="19" extent="1-1"/>
+<wire x1="43.18" y1="36.27" x2="49.53" y2="36.27" width="0" layer="19" extent="1-1"/>
+<wire x1="40.91" y1="24.13" x2="43.18" y2="36.27" width="0" layer="19" extent="1-1"/>
 <wire x1="44.685" y1="20.83" x2="40.91" y2="24.13" width="0" layer="19" extent="1-1"/>
 <wire x1="48.26" y1="17.78" x2="44.685" y2="20.83" width="0" layer="19" extent="1-1"/>
@@
 <wire x1="55.88" y1="25.71" x2="51.835" y2="20.83" width="0" layer="19" extent="1-1"/>
 <wire x1="61.87" y1="10.16" x2="52.07" y2="10.43" width="0" layer="19" extent="1-1"/>
-<wire x1="23.86" y1="35.56" x2="43.18" y2="34.02" width="0" layer="19" extent="1-1"/>
-<wire x1="23.86" y1="41.91" x2="23.86" y2="35.56" width="0" layer="19" extent="1-1"/>
-<wire x1="15.24" y1="44.18" x2="23.86" y2="41.91" width="0" layer="19" extent="1-1"/>
+<wire x1="26.11" y1="35.56" x2="43.18" y2="36.27" width="0" layer="19" extent="1-1"/>
+<wire x1="26.11" y1="41.91" x2="26.11" y2="35.56" width="0" layer="19" extent="1-1"/>
+<wire x1="15.24" y1="44.18" x2="26.11" y2="41.91" width="0" layer="19" extent="1-1"/>
 <wire x1="11.94" y1="40.405" x2="15.24" y2="44.18" width="0" layer="19" extent="1-1"/>
 <wire x1="8.89" y1="36.83" x2="11.94" y2="40.405" width="0" layer="19" extent="1-1"/>
@@
 <wire x1="17.22" y1="50.8" x2="15.24" y2="44.18" width="0" layer="19" extent="1-1"/>
 <wire x1="2.54" y1="50.08" x2="1.54" y2="38.1" width="0" layer="19" extent="1-1"/>
-<wire x1="26.4" y1="5.08" x2="46.99" y2="10.43" width="0" layer="19" extent="1-1"/>
-<wire x1="18.05" y1="7.62" x2="26.4" y2="5.08" width="0" layer="19" extent="1-1"/>
+<wire x1="27.67" y1="7.62" x2="46.99" y2="10.43" width="0" layer="19" extent="1-1"/>
+<wire x1="16.78" y1="10.16" x2="27.67" y2="7.62" width="0" layer="19" extent="1-1"/>
 </signal>
 <signal name="+3V3">
@@
 <wire x1="1.27" y1="42.91" x2="11.94" y2="38.455" width="0" layer="19" extent="1-1"/>
 <wire x1="20.955" y1="10" x2="23.82" y2="29.21" width="0" layer="19" extent="1-1"/>
-<wire x1="20.05" y1="7.62" x2="20.955" y2="10" width="0" layer="19" extent="1-1"/>
+<wire x1="18.78" y1="10.16" x2="20.955" y2="10" width="0" layer="19" extent="1-1"/>
 </signal>
 <signal name="N$34">
@@
 <wire x1="22.225" y1="10" x2="23.495" y2="10" width="0" layer="19" extent="1-1"/>
 <wire x1="21.86" y1="7.62" x2="22.225" y2="10" width="0" layer="19" extent="1-1"/>
-<wire x1="20.59" y1="5.08" x2="21.86" y2="7.62" width="0" layer="19" extent="1-1"/>
+<wire x1="21.86" y1="5.08" x2="21.86" y2="7.62" width="0" layer="19" extent="1-1"/>
 </signal>
 <signal name="VREF">
@@
 <wire x1="23.86" y1="7.62" x2="51.835" y2="14.73" width="0" layer="19" extent="1-1"/>
 <wire x1="24.765" y1="10" x2="23.86" y2="7.62" width="0" layer="19" extent="1-1"/>
-<wire x1="24.4" y1="5.08" x2="23.86" y2="7.62" width="0" layer="19" extent="1-1"/>
-<wire x1="22.59" y1="5.08" x2="24.4" y2="5.08" width="0" layer="19" extent="1-1"/>
+<wire x1="25.67" y1="7.62" x2="23.86" y2="7.62" width="0" layer="19" extent="1-1"/>
+<wire x1="23.86" y1="5.08" x2="25.67" y2="7.62" width="0" layer="19" extent="1-1"/>
 <wire x1="5.84" y1="33.255" x2="24.765" y2="10" width="0" layer="19" extent="1-1"/>
 </signal>
@@
 <contactref element="U$1" pad="17"/>
 <contactref element="R4" pad="1"/>
-<wire x1="49.235" y1="20.83" x2="49.53" y2="32.02" width="0" layer="19" extent="1-1"/>
+<wire x1="49.235" y1="20.83" x2="49.53" y2="29.77" width="0" layer="19" extent="1-1"/>
 </signal>
 <signal name="N$35">
 <contactref element="U$1" pad="20"/>
 <contactref element="R5" pad="1"/>
-<wire x1="47.285" y1="20.83" x2="43.18" y2="32.02" width="0" layer="19" extent="1-1"/>
+<wire x1="47.285" y1="20.83" x2="43.18" y2="29.77" width="0" layer="19" extent="1-1"/>
 </signal>
 <signal name="N$38">
 <contactref element="U$2" pad="17"/>
 <contactref element="R6" pad="1"/>
-<wire x1="11.94" y1="35.855" x2="21.86" y2="35.56" width="0" layer="19" extent="1-1"/>
+<wire x1="11.94" y1="35.855" x2="19.61" y2="35.56" width="0" layer="19" extent="1-1"/>
 </signal>
 <signal name="N$40">
 <contactref element="U$2" pad="20"/>
 <contactref element="R7" pad="1"/>
-<wire x1="11.94" y1="37.805" x2="21.86" y2="41.91" width="0" layer="19" extent="1-1"/>
+<wire x1="11.94" y1="37.805" x2="19.61" y2="41.91" width="0" layer="19" extent="1-1"/>
 </signal>
 </signals>
